File: ud29/ud29.kicad_sch (KiCad schematic)
At the start: 123 parts, among them J1 24V DC, J10 Conn_01x01, J11 Conn_01x01, J12 Conn_01x01, J13 Conn_01x01, J14 Conn_01x02, J15 Conn_01x03, J16 Conn_01x02, J17 Conn_01x02, J18 Conn_01x02, J19 Over Current, J2 24V AC, J3 Feedback, J4 Lead Inductor, J5 OCD, J6 Conn_02x03_Odd_Even, J7 Conn_01x02, J8 Conn_01x02, J9 Conn_01x03, Q1 IRF9540N, Q2 IRF540N, Q3 IRF9540N, Q4 IRF540N, Q5 2N3906, U1 LM7824, U15 MC34164, U2 LM7812, U3 LM7805, U4 TL3116, U5 74HC08, U6 LM311, U7 74HC74, U8 74HC14, U9 UCC27243

Commit message: minor changes
Connections:
- net +12V: now also U2.3 (VO)
- net ~PHASE: now reaches U4.8 (~{Q}), U5.1
- net EN: now reaches U5.12, U5.2, U7.9 (Q)
- net PHASE: now reaches C11.1, J16.2 (Pin_2), R16.2, U4.7 (Q), U5.13, U7.11 (Cp)
Other:
- note added: "Interrupt input"
- note added: "Over current & Under voltage protection"
- note added: "Phase alignment"
- note added: "Pulse skip & Interrupt handling"
- note added: "Voltage regulators"
- note removed: "interrupter recivers"
- note removed: "over current protection"
- note removed: "phase alignment"
- note removed: "voltage regulators"
- moved on the sheet: C18, C19, C21, C22, C23, C24, C25, C26, C27, C28, C33, C34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
